File: hdw/CH9141K/CH9141K.kicad_pcb (KiCad board)
At the start: 2 copper layers, 34.3 x 19.3 mm, 4 parts, among them U1 CH9141K

Commit message: poc - schematic & pcb for CH9141K
Parts:
- added J1: Conn_01x04, Connector_PinHeader_2.54mm:PinHeader_1x04_P2.54mm_Vertical, F.Cu at (106.0, 109.9)
- added Y1: 32M, Crystal:Crystal_SMD_5032-2Pin_5.0x3.2mm_HandSoldering, F.Cu at (91.2, 107.2)
- AE1: footprint RF_Antenna:Texas_SWRA117D_2.4GHz_Left -> RF_Antenna:Texas_SWRA117D_2.4GHz_Right
- moved C2 9.99 mm to (93.3, 120.7), turned to 0 degrees
- moved AE1 9.23 mm to (79.5, 118.2)
- moved C1 4.27 mm to (99.7, 111.5), turned to -90 degrees
- moved U1 1.47 mm to (92.7, 113.7), turned to -90 degrees
Connections:
- AE1 pad 2: (no net) -> GND
- U1 pad 1: SLEEP -> unconnected-(U1-Sleep-Pad1)
- U1 pad 10: AT -> GND
Routing:
- net RXD: track 0.00 -> 14.5 mm
- net TXD: track 0.00 -> 13.5 mm
- net VCC: track 0.00 -> 13.2 mm
- net Net-(AE1-A): track 0.00 -> 12.7 mm
- net Net-(U1-X32MO): track 0.00 -> 5.35 mm
- net Net-(U1-X32MI): track 0.00 -> 5.31 mm
- net Net-(U1-VINTA): track 0.00 -> 4.14 mm
Other:
- board text added: "GND"
- board text added: "RXD"
- board text added: "TXD"
- board text added: "V3"

Commit message: update pcb design
Routing:
- net TXD: track 13.5 -> 15.1 mm
- net RXD: track 14.5 -> 15.7 mm
- net GND: vias 0 -> 37
Other:
- board text added: "CH9141"
- board text added: "V1 2024/03"
- board text added: "nstrappazzonc"

Commit message: wip
Parts:
- removed AE1: Antenna, RF_Antenna:Texas_SWRA117D_2.4GHz_Right
- removed J1: Conn_01x04, Connector_PinHeader_2.54mm:PinHeader_1x04_P2.54mm_Vertical
- added AE2: Antenna_Shield, RF_Antenna:Texas_SWRA117D_2.4GHz_Right, F.Cu at (72.4, 118.8)
- added H1: MountingHole, MountingHole:MountingHole_3.2mm_M3, F.Cu at (76.2, 104.1)
- added H2: MountingHole, MountingHole:MountingHole_3.2mm_M3, F.Cu at (109.2, 104.1)
- added H3: MountingHole, MountingHole:MountingHole_3.2mm_M3, F.Cu at (109.2, 124.5)
- added H4: MountingHole, MountingHole:MountingHole_3.2mm_M3, F.Cu at (76.2, 124.5)
- added J2: Conn_01x03, Connector_PinHeader_2.54mm:PinHeader_1x03_P2.54mm_Vertical, F.Cu at (109.2, 111.8)
- added J3: Conn_01x04, Connector_PinHeader_2.54mm:PinHeader_1x04_P2.54mm_Vertical, F.Cu at (96.5, 127.0)
- moved C1 4.99 mm to (101.0, 106.7), turned to 90 degrees
- moved C2 4.49 mm to (88.9, 121.3), turned to -90 degrees
- moved U1 0.63 mm to (92.7, 114.3)
- moved Y1 0.51 mm to (91.2, 106.7)
Connections:
- U1 pad 10: GND -> AT
Routing:
- net VCC: track 13.2 -> 50.4 mm
- net AT: track 0.00 -> 15.7 mm
- net Net-(AE2-A): track 12.7 -> 19.0 mm
- net RXD: track 15.7 -> 10.4 mm
- net TXD: track 15.1 -> 9.96 mm
- net GND: vias 37 -> 35
Other:
- board size 34.3 x 19.3 mm -> 47 x 27.9 mm
- board text added: "AT"
- board text added: "CH9141K"
- board text added: "RX"
- board text added: "TX"
- board text added: "V1.1 2024-04"
- board text added: "nicola@strappazzon.me"
- board text removed: "CH9141"
- board text removed: "RXD"
- board text removed: "TXD"
- board text removed: "V1 2024/03"
- board text removed: "nstrappazzonc"
